File: hardware/electrical/sd.kicad_sch (KiCad schematic)
At the start: 9 parts, among them J3 Micro_SD_Card_Det

Commit message: Footprint assignment
Parts:
- C35: footprint (none) -> Capacitor_SMD:C_0603_1608Metric
- C36: footprint (none) -> Capacitor_SMD:C_0402_1005Metric
- J3: footprint (none) -> Connector_Card:microSD_HC_Molex_104031-0811
- R13, R14, R15, R16, R17, R18: footprint (none) -> Resistor_SMD:R_0402_1005Metric
Changed lines of the file:
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@@
       (effects (font (size 1.27 1.27)) (justify left))
     )
-    (property "Footprint" "" (id 2) (at 103.632 92.71 90)
+    (property "Footprint" "Resistor_SMD:R_0402_1005Metric" (id 2) (at 103.632 92.71 90)
       (effects (font (size 1.27 1.27)) hide)
     )
@@
       (effects (font (size 1.27 1.27)) (justify left))
     )
-    (property "Footprint" "" (id 2) (at 121.412 92.71 90)
+    (property "Footprint" "Resistor_SMD:R_0402_1005Metric" (id 2) (at 121.412 92.71 90)
       (effects (font (size 1.27 1.27)) hide)
     )
@@
       (effects (font (size 1.27 1.27)) (justify left))
     )
-    (property "Footprint" "" (id 2) (at 130.302 92.71 90)
+    (property "Footprint" "Resistor_SMD:R_0402_1005Metric" (id 2) (at 130.302 92.71 90)
       (effects (font (size 1.27 1.27)) hide)
     )
@@
       (effects (font (size 1.27 1.27)) (justify left))
     )
-    (property "Footprint" "" (id 2) (at 135.5852 67.31 0)
+    (property "Footprint" "Capacitor_SMD:C_0603_1608Metric" (id 2) (at 135.5852 67.31 0)
       (effects (font (size 1.27 1.27)) hide)
     )
@@
       (effects (font (size 1.27 1.27)) (justify left))
     )
-    (property "Footprint" "" (id 2) (at 148.2852 67.31 0)
+    (property "Footprint" "Capacitor_SMD:C_0402_1005Metric" (id 2) (at 148.2852 67.31 0)
       (effects (font (size 1.27 1.27)) hide)
     )
@@
       (effects (font (size 1.27 1.27)) (justify left))
     )
-    (property "Footprint" "" (id 2) (at 112.522 92.71 90)
+    (property "Footprint" "Resistor_SMD:R_0402_1005Metric" (id 2) (at 112.522 92.71 90)
       (effects (font (size 1.27 1.27)) hide)
     )
@@
       (effects (font (size 1.27 1.27)) hide)
     )
-    (property "Footprint" "" (id 2) (at 234.95 91.44 0)
+    (property "Footprint" "Connector_Card:microSD_HC_Molex_104031-0811" (id 2) (at 234.95 91.44 0)
       (effects (font (size 1.27 1.27)) hide)
     )
@@
       (effects (font (size 1.27 1.27)) (justify left))
     )
-    (property "Footprint" "" (id 2) (at 148.082 92.71 90)
+    (property "Footprint" "Resistor_SMD:R_0402_1005Metric" (id 2) (at 148.082 92.71 90)
       (effects (font (size 1.27 1.27)) hide)
     )
@@
       (effects (font (size 1.27 1.27)) (justify left))
     )
-    (property "Footprint" "" (id 2) (at 139.192 92.71 90)
-      (effects (font (size 1.27 1.27)) hide)
-    )
+    (property "Footprint" "Resistor_SMD:R_0402_1005Metric" (id 2) (at 139.192 92.71 90)
+      (effects (font (size 1.27 1.27)) hide)
+    )
