File: hardware/electrical/sd.kicad_sch (KiCad schematic)
At the start: 9 parts, among them J3 Micro_SD_Card_Det

Commit message: PCB Rev 1.0
Parts:
- C35: value 4u7 -> 10u; footprint Capacitor_SMD:C_0402_1005Metric -> Capacitor_SMD:C_1206_3216Metric; LCSC Part # (none) -> C7171; Mfr (none) -> Kyocera AVX; Mfr. Part # (none) -> TAJA106K016RNJ
- C36: LCSC Part # (none) -> C30274; Mfr (none) -> FH(Guangdong Fenghua Advanced Tech); Mfr. Part # (none) -> 0402CG6R0C500NT
- J3: footprint Connector_Card:microSD_HC_Molex_104031-0811 -> (none); LCSC Part # (none) -> C381084; Mfr (none) -> XKB Connectivity; Mfr. Part # (none) -> XKTF-N02-N
- R13, R14, R15, R16, R17, R18: LCSC Part # (none) -> C25744; Mfr (none) -> UNI-ROYAL(Uniroyal Elec); Mfr. Part # (none) -> 0402WGF1002TCE
Connections:
- net +3V3 renamed VDD
