File: hardware/electrical/usb.kicad_sch (KiCad schematic)
At the start: 15 parts, among them J1 USB_B_Micro, U1 USB3300-EZK

Commit message: Component selection
Parts:
- C1: value 100u -> 10u; LCSC Part # (none) -> C15525; Mfr (none) -> Samsung Electro-Mechanics; Mfr. Part # (none) -> CL05A106MQ5NUNC
- C2, C3, C4, C5: footprint (none) -> Capacitor_SMD:C_0402_1005Metric; LCSC Part # (none) -> C1525; Mfr (none) -> Samsung Electro-Mechanics; Mfr. Part # (none) -> CL05B104KO5NNNC
- C6, C7, C8: footprint (none) -> Capacitor_SMD:C_0402_1005Metric; LCSC Part # (none) -> C23733; Mfr (none) -> Samsung Electro-Mechanics; Mfr. Part # (none) -> CL05A475MP5NRNC
- D1: footprint (none) -> Diode_SMD:D_SOD-123F; LCSC Part # (none) -> C2990473; Mfr (none) -> Liown; Mfr. Part # (none) -> SMF6.0CA
- FB1: footprint Diode_SMD:D_0201_0603Metric -> Inductor_SMD:L_0805_2012Metric; LCSC Part # (none) -> C1017; Mfr (none) -> Sunlord; Mfr. Part # (none) -> GZ2012D601TF
- J1: footprint (none) -> Connector_USB:USB_Micro-B_Amphenol_10118194_Horizontal; LCSC Part # (none) -> C132563; Mfr (none) -> Amphenol ICC; Mfr. Part # (none) -> 10118194-0001LF
- R1: value 670R -> 680R; footprint (none) -> Resistor_SMD:R_0402_1005Metric; LCSC Part # (none) -> C25130; Mfr (none) -> UNI-ROYAL(Uniroyal Elec); Mfr. Part # (none) -> 0402WGF6800TCE
- R2: footprint (none) -> Resistor_SMD:R_0402_1005Metric; LCSC Part # (none) -> C25752; Mfr (none) -> UNI-ROYAL(Uniroyal Elec); Mfr. Part # (none) -> 0402WGF1202TCE
- R3: footprint (none) -> Resistor_SMD:R_0402_1005Metric; LCSC Part # (none) -> C25105; Mfr (none) -> UNI-ROYAL(Uniroyal Elec); Mfr. Part # (none) -> 0402WGF330JTCE
- U1: LCSC Part # (none) -> C108383; Mfr (none) -> Microchip Tech; Mfr. Part # (none) -> USB3300-EZK-TR
