File: hardware/electrical/usb.kicad_sch (KiCad schematic)
At the start: 15 parts, among them J1 USB_B_Micro, U1 USB3300-EZK

Commit message: Route ULPI and power supply
Connections:
- net +3V3 is gone; now on net VDD: U1.31 (REG_EN)
Changed lines of the file:
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@@
   (junction (at 170.18 48.26) (diameter 0) (color 0 0 0 0)
+  )
+  (junction (at 203.2 114.3) (diameter 0) (color 0 0 0 0)
   )
   (junction (at 139.7 66.04) (diameter 0) (color 0 0 0 0)
@@
     (stroke (width 0) (type default))
   )
+  (wire (pts (xy 203.2 114.3) (xy 205.74 114.3))
+    (stroke (width 0) (type default))
+  )
   (wire (pts (xy 90.17 73.66) (xy 90.17 83.82))
     (stroke (width 0) (type default))
@@
     (stroke (width 0) (type default))
   )
+  (wire (pts (xy 203.2 111.76) (xy 203.2 114.3))
+    (stroke (width 0) (type default))
+  )
   (wire (pts (xy 190.5 50.8) (xy 190.5 48.26))
     (stroke (width 0) (type default))
@@
     (stroke (width 0) (type default))
   )
-  (wire (pts (xy 165.1 114.3) (xy 205.74 114.3))
+  (wire (pts (xy 165.1 114.3) (xy 203.2 114.3))
     (stroke (width 0) (type default))
   )
@@
     )
   )
+  (netclass_flag "" (length 2.54) (shape round) (at 203.2 111.76 0)
+    (effects (font (size 1.27 1.27)) (justify left bottom))
+    (property "Netclass" "ULPI" (at 203.2 106.68 0)
+      (effects (font (size 1.27 1.27) italic))
+    )
+  )
   (netclass_flag "" (length 2.54) (shape round) (at 90.17 73.66 0)
     (effects (font (size 1.27 1.27)) (justify left bottom))
@@
         (path "/7363a4f0-2da1-4086-abed-ea6709c3a185/b2a90f2c-c4bd-40df-ad3c-0b37c5fa6b32"
           (reference "#FLG01") (unit 1)
-        )
-      )
-    )
-  )
-  (symbol (lib_id "power:+3V3") (at 116.84 106.68 0) (unit 1)
-    (in_bom yes) (on_board yes) (dnp no) (fields_autoplaced)
-    (property "Reference" "#PWR04" (at 116.84 110.49 0)
-      (effects (font (size 1.27 1.27)) hide)
-    )
-    (property "Value" "+3V3" (at 116.84 101.6 0)
-      (effects (font (size 1.27 1.27)))
-    )
-    (property "Footprint" "" (at 116.84 106.68 0)
-      (effects (font (size 1.27 1.27)) hide)
-    )
-    (property "Datasheet" "" (at 116.84 106.68 0)
-      (effects (font (size 1.27 1.27)) hide)
-    )
-    (pin "1")
-    (instances
-      (project "3885"
-        (path "/7363a4f0-2da1-4086-abed-ea6709c3a185/b2a90f2c-c4bd-40df-ad3c-0b37c5fa6b32"
-          (reference "#PWR04") (unit 1)
         )
       )
@@
         )
       )
+    )
+  )
+  (symbol (lib_id "power:VDD") (at 116.84 106.68 0) (unit 1)
+    (in_bom yes) (on_board yes) (dnp no) (fields_autoplaced)
+    (property "Reference" "#PWR04" (at 116.84 110.49 0)
+      (effects (font (size 1.27 1.27)) hide)
+    )
+    (property "Value" "VDD" (at 116.84 102.87 0)
+      (effects (font (size 1.27 1.27)))
+    )
+    (property "Footprint" "" (at 116.84 106.68 0)
+      (effects (font (size 1.27 1.27)) hide)
+    )
+    (property "Datasheet" "" (at 116.84 106.68 0)
+      (effects (font (size 1.27 1.27)) hide)
+    )
+    (pin "1")
+    (instances
+      (project "3885"
+        (path "/7363a4f0-2da1-4086-abed-ea6709c3a185/b2a90f2c-c4bd-40df-ad3c-0b37c5fa6b32"
+          (reference "#PWR04") (unit 1)
+        )
+      )

Commit message: Replace USB connector with SMD part
Parts:
- J1: footprint Connector_USB:USB_Micro-B_Amphenol_10118194_Horizontal -> Connector_USB:USB_Micro-B_Amphenol_10104110_Horizontal; LCSC Part # C132563 -> C2931352; Mfr. Part # 10118194-0001LF -> 10104110-0001LF
Changed lines of the file:
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@@
       (effects (font (size 1.27 1.27)) hide)
     )
-    (property "Footprint" "Connector_USB:USB_Micro-B_Amphenol_10118194_Horizontal" (at 38.1 82.55 0)
+    (property "Footprint" "Connector_USB:USB_Micro-B_Amphenol_10104110_Horizontal" (at 38.1 82.55 0)
       (effects (font (size 1.27 1.27)) hide)
     )
@@
       (effects (font (size 1.27 1.27)) hide)
     )
-    (property "LCSC Part #" "C132563" (at 34.29 81.28 0)
+    (property "LCSC Part #" "C2931352" (at 34.29 81.28 0)
       (effects (font (size 1.27 1.27)) hide)
     )
@@
       (effects (font (size 1.27 1.27)) hide)
     )
-    (property "Mfr. Part #" "10118194-0001LF" (at 34.29 81.28 0)
+    (property "Mfr. Part #" "10104110-0001LF" (at 34.29 81.28 0)
       (effects (font (size 1.27 1.27)) hide)
     )

Commit message: JLCPCB position and rotation adjustments
Parts:
- U1: footprint Package_DFN_QFN:QFN-32-1EP_5x5mm_P0.5mm_EP3.45x3.45mm -> 3885:JLC_QFN-32-1EP_5x5mm_P0.5mm_EP3.45x3.45mm
Changed lines of the file:
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@@
       (effects (font (size 1.27 1.27)) (justify left))
     )
-    (property "Footprint" "Package_DFN_QFN:QFN-32-1EP_5x5mm_P0.5mm_EP3.45x3.45mm" (at 177.8 128.27 0)
+    (property "Footprint" "3885:JLC_QFN-32-1EP_5x5mm_P0.5mm_EP3.45x3.45mm" (at 177.8 128.27 0)
       (effects (font (size 1.27 1.27)) hide)
     )
