File: hardware/electrical/3885.kicad_pcb (KiCad board)
At the start: 4 copper layers, 33 x 77 mm, 112 parts, among them J1 USB_B_Micro, J2 TC2030, J3 Micro_SD_Card_Det1, J4 JST-PH, J5 FFC, Q1 AO3400A, Q2 AO3400A, Q3 AO3401A, Q4 AO3401A, Q5 2N7002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

Commit message: Connect U5 VSS to -BATT instead of GND
Connections:
- U5 pad 6: GND -> -BATT
Routing:
- net -BATT: track 15.0 -> 17.8 mm
- net GND: track 118.2 -> 116.0 mm, vias 435 -> 434
Changed lines of the file:
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@@
       (net 132 "Net-(#FLG03-pwr)") (pinfunction "VDD") (pintype "power_in"))
     (pad "6" smd roundrect (at 1.1375 -0.95 270) (size 1.325 0.6) (layers "F.Cu" "F.Paste" "F.Mask") (roundrect_rratio 0.25)
-      (net 1 "GND") (pinfunction "VSS") (pintype "power_in"))
+      (net 3 "-BATT") (pinfunction "VSS") (pintype "power_in"))
     (model "${KICAD6_3DMODEL_DIR}/Package_TO_SOT_SMD.3dshapes/SOT-23-6.wrl"
       (offset (xyz 0 0 0))
@@
   (segment (start 150 76.21) (end 150.95 76.21) (width 0.5) (layer "F.Cu") (net 1))
   (segment (start 138.25 135.4375) (end 138.25 135.85) (width 0.25) (layer "F.Cu") (net 1))
-  (segment (start 152.95 104.4) (end 152.325 103.775) (width 0.25) (layer "F.Cu") (net 1))
   (segment (start 160.425 114.475) (end 160.4 114.45) (width 0.25) (layer "F.Cu") (net 1))
   (segment (start 154.25 125.775) (end 154.25 124.6) (width 0.25) (layer "F.Cu") (net 1))
@@
   (segment (start 161.95 76.75) (end 163.04 76.75) (width 0.5) (layer "F.Cu") (net 1))
   (segment (start 138.27 122.1) (end 138.27 123.1) (width 0.25) (layer "F.Cu") (net 1))
-  (segment (start 152.325 103.775) (end 151.6 103.775) (width 0.25) (layer "F.Cu") (net 1))
   (segment (start 148.5 101.675) (end 148.5 100.75) (width 0.5) (layer "F.Cu") (net 1))
   (segment (start 138.27 118.85) (end 138.27 119.53) (width 0.25) (layer "F.Cu") (net 1))
@@
   (segment (start 147.25 72.8) (end 147.25 74.35) (width 0.25) (layer "F.Cu") (net 1))
   (segment (start 136.75 116.8) (end 136.75 115.15) (width 0.25) (layer "F.Cu") (net 1))
-  (segment (start 152.95 104.75) (end 152.95 104.4) (width 0.25) (layer "F.Cu") (net 1))
   (segment (start 154.8 88.87) (end 155.8 88.87) (width 0.5) (layer "F.Cu") (net 1))
   (segment (start 149 76.21) (end 149 77.05) (width 0.5) (layer "F.Cu") (net 1))
@@
   (segment (start 147.5 142.05) (end 149.5 142.05) (width 0.5) (layer "F.Cu") (net 1))
   (segment (start 143 126.85) (end 143 127.43) (width 0.25) (layer "F.Cu") (net 1))
-  (segment (start 151.6 103.775) (end 151.425 103.6) (width 0.25) (layer "F.Cu") (net 1))
   (segment (start 156.35 102.75) (end 155.725 102.125) (width 0.5) (layer "F.Cu") (net 1))
   (segment (start 138.27 114.6) (end 138.27 113.6) (width 0.25) (layer "F.Cu") (net 1))
@@
   (via (at 152 138.5) (size 0.46) (drill 0.2) (layers "F.Cu" "B.Cu") (net 1))
   (via (at 160 139.5) (size 0.46) (drill 0.2) (layers "F.Cu" "B.Cu") (net 1))
-  (via (at 151.425 103.6) (size 0.46) (drill 0.2) (layers "F.Cu" "B.Cu") (net 1))
   (via (at 148 118.5) (size 0.46) (drill 0.2) (layers "F.Cu" "B.Cu") (net 1))
   (via (at 164 101.5) (size 0.46) (drill 0.2) (layers "F.Cu" "B.Cu") (net 1))
@@
   (segment (start 154.37 106.25) (end 153.41 106.25) (width 0.5) (layer "F.Cu") (net 2))
   (segment (start 164.45 109.6) (end 162.2 107.35) (width 0.5) (layer "F.Cu") (net 3))
+  (segment (start 154.68 104.5) (end 153.2 104.5) (width 0.25) (layer "F.Cu") (net 3))
+  (segment (start 153.2 104.5) (end 152.95 104.75) (width 0.25) (layer "F.Cu") (net 3))
+  (segment (start 155.33 105.15) (end 154.68 104.5) (width 0.25) (layer "F.Cu") (net 3))
   (segment (start 161.2 105.15) (end 162.2 106.15) (width 0.5) (layer "F.Cu") (net 3))
   (segment (start 162.2 106.15) (end 162.2 107.35) (width 0.5) (layer "F.Cu") (net 3))
